File: fonteDC/_saved_fonteDC.sch (KiCad schematic (older format))
At the start: 18 parts, among them J1 Conn_01x02, T1 Transformer_1P_SS, U1 LM7805_TO220

Commit message: Tudo antes dos footprints dos capacitores e transformador
Parts:
- AC_in1: footprint (none) -> fonteDC:AC_in
- Cc1, Cc2: footprint (none) -> fonteDC:C_Disc_D5.0mm_W2.5mm_P5.00mm
- D1, D2, D3, D4: footprint (none) -> fonteDC:D_5W_P12.70mm_Horizontal
- D5, D6: footprint (none) -> fonteDC:LED_D8.0mm
- F1: footprint (none) -> fonteDC:Fuseholder5x20_horiz_SemiClosed_Casing10x25mm
- R1, R2: footprint (none) -> fonteDC:R_Axial_DIN0204_L3.6mm_D1.6mm_P7.62mm_Horizontal
- U1: footprint TO_SOT_Packages_THT:TO-220_Vertical -> fonteDC:TO-220-3_Vertical
Connections:
- net GND: now also T1.5 (SB), switch1.4 (GND220), switch1.6 (GND110)
Changed lines of the file:
@@
 F 0 "AC_in1" H 900 3250 60  0000 C CNN
 F 1 "AC_in" H 900 3350 60  0000 C CNN
-F 2 "" H 900 3250 60  0001 C CNN
+F 2 "fonteDC:AC_in" H 900 3250 60  0001 C CNN
 F 3 "" H 900 3250 60  0001 C CNN
 	1    1250 3250
@@
 F 0 "F1" V 1330 3900 50  0000 C CNN
 F 1 "Fuse" V 1175 3900 50  0000 C CNN
-F 2 "" V 1180 3900 50  0001 C CNN
+F 2 "fonteDC:Fuseholder5x20_horiz_SemiClosed_Casing10x25mm" V 1180 3900 50  0001 C CNN
 F 3 "" H 1250 3900 50  0001 C CNN
 	1    1250 3900
@@
 F 0 "R1" V 5480 3100 50  0000 C CNN
 F 1 "R" V 5400 3100 50  0000 C CNN
-F 2 "" V 5330 3100 50  0001 C CNN
+F 2 "fonteDC:R_Axial_DIN0204_L3.6mm_D1.6mm_P7.62mm_Horizontal" V 5330 3100 50  0001 C CNN
 F 3 "" H 5400 3100 50  0001 C CNN
 	1    5400 3100
@@
 F 0 "D5" H 5400 3650 50  0000 C CNN
 F 1 "LED" H 5400 3450 50  0000 C CNN
-F 2 "" H 5400 3550 50  0001 C CNN
+F 2 "fonteDC:LED_D8.0mm" H 5400 3550 50  0001 C CNN
 F 3 "" H 5400 3550 50  0001 C CNN
 	1    5400 3550
@@
 F 0 "D1" H 6100 2850 50  0000 C CNN
 F 1 "D" H 6100 2650 50  0000 C CNN
-F 2 "" H 6100 2750 50  0001 C CNN
+F 2 "fonteDC:D_5W_P12.70mm_Horizontal" H 6100 2750 50  0001 C CNN
 F 3 "" H 6100 2750 50  0001 C CNN
 	1    6100 2750
@@
 F 0 "D2" H 6100 4050 50  0000 C CNN
 F 1 "D" H 6100 3850 50  0000 C CNN
-F 2 "" H 6100 3950 50  0001 C CNN
+F 2 "fonteDC:D_5W_P12.70mm_Horizontal" H 6100 3950 50  0001 C CNN
 F 3 "" H 6100 3950 50  0001 C CNN
 	1    6100 3950
@@
 F 0 "D3" H 6450 3250 50  0000 C CNN
 F 1 "D" H 6450 3050 50  0000 C CNN
-F 2 "" H 6450 3150 50  0001 C CNN
+F 2 "fonteDC:D_5W_P12.70mm_Horizontal" H 6450 3150 50  0001 C CNN
 F 3 "" H 6450 3150 50  0001 C CNN
 	1    6450 3150
@@
 F 0 "D4" H 6450 3700 50  0000 C CNN
 F 1 "D" H 6450 3500 50  0000 C CNN
-F 2 "" H 6450 3600 50  0001 C CNN
+F 2 "fonteDC:D_5W_P12.70mm_Horizontal" H 6450 3600 50  0001 C CNN
 F 3 "" H 6450 3600 50  0001 C CNN
 	1    6450 3600
@@
 F 0 "Cc1" H 7675 3500 50  0000 L CNN
 F 1 "C" H 7675 3300 50  0000 L CNN
-F 2 "" H 7688 3250 50  0001 C CNN
+F 2 "fonteDC:C_Disc_D5.0mm_W2.5mm_P5.00mm" H 7688 3250 50  0001 C CNN
 F 3 "" H 7650 3400 50  0001 C CNN
 	1    7650 3400
@@
 F 0 "U1" H 8150 2875 50  0000 C CNN
 F 1 "LM7805_TO220" H 8300 2875 50  0000 L CNN
-F 2 "TO_SOT_Packages_THT:TO-220_Vertical" H 8300 2975 50  0001 C CIN
+F 2 "fonteDC:TO-220-3_Vertical" H 8300 2975 50  0001 C CIN
 F 3 "" H 8300 2700 50  0001 C CNN
 	1    8300 2750
@@
 F 0 "Cc2" H 9275 3500 50  0000 L CNN
 F 1 "C" H 9275 3300 50  0000 L CNN
-F 2 "" H 9288 3250 50  0001 C CNN
+F 2 "fonteDC:C_Disc_D5.0mm_W2.5mm_P5.00mm" H 9288 3250 50  0001 C CNN
 F 3 "" H 9250 3400 50  0001 C CNN
 	1    9250 3400
@@
 F 0 "R2" V 9780 3050 50  0000 C CNN
 F 1 "R" V 9700 3050 50  0000 C CNN
-F 2 "" V 9630 3050 50  0001 C CNN
+F 2 "fonteDC:R_Axial_DIN0204_L3.6mm_D1.6mm_P7.62mm_Horizontal" V 9630 3050 50  0001 C CNN
 F 3 "" H 9700 3050 50  0001 C CNN
 	1    9700 3050
@@
 F 0 "D6" H 9700 3600 50  0000 C CNN
 F 1 "LED" H 9700 3400 50  0000 C CNN
-F 2 "" H 9700 3500 50  0001 C CNN
+F 2 "fonteDC:LED_D8.0mm" H 9700 3500 50  0001 C CNN
 F 3 "" H 9700 3500 50  0001 C CNN
 	1    9700 3500
@@
 Wire Wire Line
 	3850 3550 4000 3550
+Wire Wire Line
+	3750 3700 3750 3650
+Connection ~ 3750 3650
 $EndSCHEMATC

Commit message: Adicionando capacitores e porta fusível
Parts:
- Ce1: footprint (none) -> fonteDC:CP_elet_7mF
- Ce2: footprint (none) -> fonteDC:CP_elet_10mF
Changed lines of the file:
@@
 F 0 "Ce1" H 7375 3500 50  0000 L CNN
 F 1 "CP1" H 7375 3300 50  0000 L CNN
-F 2 "" H 7350 3400 50  0001 C CNN
+F 2 "fonteDC:CP_elet_7mF" H 7350 3400 50  0001 C CNN
 F 3 "" H 7350 3400 50  0001 C CNN
 	1    7350 3400
@@
 F 0 "Ce2" H 8925 3500 50  0000 L CNN
 F 1 "CP1" H 8925 3300 50  0000 L CNN
-F 2 "" H 8900 3400 50  0001 C CNN
+F 2 "fonteDC:CP_elet_10mF" H 8900 3400 50  0001 C CNN
 F 3 "" H 8900 3400 50  0001 C CNN
 	1    8900 3400
